File: Dreadnoughtus/Dreadnoughtus.kicad_pcb (KiCad board)
At the start: 2 copper layers, 382 parts, among them U1 Elite-C, U2 PRTR5V0U2X, U3 PRTR5V0U2X

Commit message: tracked most switches and diodes
Parts:
- added D214: DIODE, Keebio-Parts:Diode-dual, F.Cu at (506.4, 295.3)
- U1: footprint Keebio-Parts:Elite-C-castellated-29pin-holes -> Keebio-Parts:Elite-C
- U3: footprint Keebio-Parts:I2C_Breakout -> Keebio-Parts:SW_Tactile_SPST_Angled_MJTP1117; moved to B.Cu
- moved R1 725.1 mm to (980.3, 270.7), turned to 180 degrees
- moved R0 712.0 mm to (980.3, 273.8), turned to 180 degrees
- moved U2 695.2 mm to (989.8, 260.0)
- moved U3 683.4 mm to (972.5, 255.3), turned to 180 degrees
- moved D0 666.5 mm to (971.5, 290.5), turned to 90 degrees
- moved D34 635.8 mm to (895.4, 404.8), turned to 90 degrees
- moved D10 628.8 mm to (990.6, 347.7), turned to 90 degrees
- moved D53 605.6 mm to (876.3, 366.7), turned to 90 degrees
- moved D11 597.4 mm to (990.6, 366.7), turned to 90 degrees
- moved D36 586.3 mm to (914.4, 309.6), turned to 90 degrees
- moved D41 584.5 mm to (914.4, 404.8), turned to 90 degrees
- moved D5 568.2 mm to (971.5, 385.8), turned to 90 degrees
- moved D54 566.7 mm to (876.3, 385.8), turned to 90 degrees
- moved D13 556.7 mm to (990.6, 404.8), turned to 90 degrees
- moved D59 549.0 mm to (819.1, 347.7), turned to 90 degrees
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Connections:
- U1 pad 10: row3 -> row2
- U1 pad 11: row4 -> row1
- U1 pad 12: row5 -> row0
- U1 pad 7: row0 -> row5
- U1 pad 8: row1 -> row4
- U1 pad 9: row2 -> row3
- U2 pad 2: SDA -> +5V
- U2 pad 4: +5V -> SDA
Routing:
- net row10: track 0.00 -> 598.1 mm, vias 0 -> 2
- net row9: track 0.00 -> 553.3 mm, vias 0 -> 2
- net row8: track 0.00 -> 551.6 mm, vias 0 -> 2
- net Net-(D105-Pad2): track 0.00 -> 523.5 mm
- net Net-(D10-Pad2): track 0.00 -> 497.0 mm
- net Net-(D103-Pad2): track 0.00 -> 496.1 mm
- net Net-(D1-Pad2): track 0.00 -> 496.0 mm
- net Net-(D104-Pad2): track 0.00 -> 495.4 mm
- net Net-(D109-Pad2): track 0.00 -> 495.4 mm
- net Net-(D107-Pad2): track 0.00 -> 494.4 mm
- net row7: track 0.00 -> 489.9 mm, vias 0 -> 3
- net Net-(D106-Pad2): track 0.00 -> 475.2 mm
- net Net-(D0-Pad2): track 0.00 -> 473.8 mm
- net Net-(D102-Pad2): track 0.00 -> 469.5 mm
- net Net-(D110-Pad2): track 0.00 -> 469.4 mm
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Other:
- board outline added: 498.5 x 159.5 mm
