File: Dreadnoughtus/Dreadnoughtus.kicad_pcb (KiCad board)
At the start: 2 copper layers, 498.5 x 156.4 mm, 383 parts, among them U1 Elite-C, U2 PRTR5V0U2X, U3 PRTR5V0U2X

Commit message: small tweak to I2C breakout position
Parts:
- moved R0 480.2 mm to (515.9, 137.9)
- moved R1 480.2 mm to (515.9, 134.8)
- moved U2 469.6 mm to (537.4, 125.4)
- moved D100 467.2 mm to (258.1, 191.9)
- moved D101 467.2 mm to (258.1, 211.0)
- moved D103 467.2 mm to (258.1, 249.1)
- moved D104 467.2 mm to (258.1, 267.9)
- moved D133 467.2 mm to (200.9, 153.8)
- moved D134 467.2 mm to (200.9, 172.9)
- moved D135 467.2 mm to (200.9, 191.9)
- moved D136 467.2 mm to (200.9, 211.0)
- moved D138 467.2 mm to (200.9, 249.1)
- moved D139 467.2 mm to (200.9, 268.1)
- moved D14 467.2 mm to (486.7, 153.8)
- moved D15 467.2 mm to (486.7, 172.9)
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Routing:
- net SDA: track 53.6 -> 64.7 mm
- net +5V: track 81.6 -> 74.3 mm
- net SCL: track 62.5 -> 58.0 mm
- net row7: track 489.9 -> 487.0 mm
- net row10: track 596.0 -> 594.3 mm
- net row3: track 319.9 -> 318.4 mm
- net GND1: track 90.5 -> 89.1 mm
- net row2: track 289.0 -> 287.8 mm
- net Net-(D84-Pad1): track 6.97 -> 5.86 mm
- net row0: track 269.4 -> 268.3 mm
- net row4: track 354.6 -> 353.5 mm
- net row9: track 548.8 -> 548.0 mm
Other:
- board size 498.5 x 156.4 mm -> 496.9 x 155.6 mm

Commit message: another final touch
Parts:
- moved D10 103.7 mm to (517.3, 110.7)
- moved D11 103.7 mm to (517.3, 129.8)
- moved D12 103.7 mm to (517.3, 148.8)
- moved D13 103.7 mm to (517.3, 167.9)
- moved D201 103.7 mm to (506.8, 57.5)
- moved D205 103.7 mm to (356.1, 132.9)
- moved D207 103.7 mm to (280.7, 171.8)
- moved D208 103.7 mm to (260.1, 171.8)
- moved D21 103.7 mm to (479.2, 53.6)
- moved D22 103.7 mm to (479.2, 72.6)
- moved D24 103.7 mm to (479.2, 110.7)
- moved D25 103.7 mm to (479.2, 129.8)
- moved D26 103.7 mm to (479.2, 148.8)
- moved D27 103.7 mm to (479.2, 167.9)
- moved D42 103.7 mm to (383.9, 53.6)
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Routing:
- net GND1: track 89.1 -> 87.7 mm
Other:
- outline, holes or cut-outs redrawn
- board text added: "github.com/KristoferKoehn/Dreadnoughtus-Catatonia"
